File: MiniFeedLid.kicad_pcb (KiCad board)
At the start: 2 copper layers, 100 x 98 mm, 3 parts

Commit message: Fixed version silkscreen
Other:
- board text added: "v1.0"
- board text removed: "V1.0"
Changed lines of the file:
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@@
     )
   )
-  (gr_text V1.0 (at 189.824999 127.725) (layer B.SilkS)
+  (gr_text v1.0 (at 189.824999 127.725) (layer B.SilkS)
     (effects (font (size 1 1) (thickness 0.15)) (justify mirror))
   )
